Commit message: fix: pipe chassis mass into URDF (#410)
* fix: pipe chassis mass into URDF

* fix: sync obstacle defaults with template

---------

Co-authored-by: Bruno Hjorth <bruno@MacBook-Pro-som-tillhor-Bruno.local>

File: ros2/src/mowgli_bringup/urdf/mowgli.urdf.xacro (robot description, xacro)
@@ -45,4 +45,5 @@
   <xacro:arg name="chassis_width"    default="0.40"/>
   <xacro:arg name="chassis_height"   default="0.19"/>
+  <xacro:arg name="chassis_mass_kg"  default="8.76"/>
   <xacro:arg name="chassis_center_x" default="0.20"/>
   <xacro:arg name="wheel_radius"     default="0.093"/>
@@ -71,5 +72,5 @@
   <xacro:property name="caster_x_offset"  value="${chassis_cx + base_length/2.0 - caster_radius}"/>
   <xacro:property name="caster_track"     value="$(arg caster_track)"/>
-  <xacro:property name="base_mass"        value="8.76"/>
+  <xacro:property name="base_mass"        value="$(arg chassis_mass_kg)"/>
   <xacro:property name="blade_radius"     value="$(arg blade_radius)"/>
   <xacro:property name="blade_height"     value="0.01"/>
